Commit message: changed angle and script

File: newbot.urdf.xacro (robot description, xacro)
@@ -32,5 +32,5 @@
   </link>
   <joint name="camera_joint" type="fixed">
-    <origin xyz="0.040 -0.011 0.130" rpy="0 0.8 0"/>
+    <origin xyz="0.040 -0.011 0.130" rpy="0 0.52 0"/>
     <parent link="base_link"/>
     <child link="camera_link"/>
